File: Board Files/SGC.0.brd (EAGLE design)
At the start: 100 x 80 mm, 1 part, among them IC1 AT90USB1287-AU

Commit message: Microcontroller block update
Parts:
- added C1: 1.0uF, SparkFun-Capacitors:0603-CAP
- added C10: 1uF, adafruit:C0603
- added C11, C9: 15pF, adafruit:C0603
- added C12, C13, C8: 0.1uF, adafruit:C0603
- added D4, D5: RED, SparkFun-LED:LED-0603
- added HWB, RESET: (no value), SparkFun-Electromechanical:TACTILE_SWITCH_SMD
- added JP1: M02PTH, SparkFun-Connectors:1X02
- added R1, R3, R35, R36: 47K, adafruit:R0603
- added R37, R38: 22, adafruit:R0603
- added R39, R40: 330, SparkFun-Resistors:0603-RES
- added U$23: S1AB-13-F, Helmet:SMB
- added X1: (no value), adafruit:CTS406
- added X3: MINI-USB-UX60-MB-5S8, con-hirose:UX60-MB-5S8
Connections:
- removed net UCAP: IC1.7
- removed net UGND: IC1.6
- new net 3.3V: C12.1, C13.1, R35.1, R36.2
- new net A6: R39.2
- new net A7: R40.2
- new net BATTSIG: R1.1, R3.2
- new net D+: R37.1
- new net D-: R38.1
- new net HWB: HWB.1, HWB.2, IC1.43, R36.1
- new net ID: X3.4
- new net N$1: R37.2, X3.3
- new net N$11: C8.1
- new net N$2: R38.2, X3.2
- new net N$29: D4.A, R39.1
- new net N$3: C10.1, IC1.7
- new net N$31: D5.A, R40.1
- new net RESET: IC1.20, R35.2, RESET.1, RESET.2
- new net VIN: C1.1, JP1.2, R1.2, U$23.M
- new net XTAL1: C11.1, X1.1
- new net XTAL2: C9.1, X1.3
- net GND: now also C1.2, C10.2, C11.2, C12.2, C13.2, C8.2, C9.2, D4.C, D5.C, HWB.3, HWB.4, IC1.6, JP1.1, R3.1, RESET.3, RESET.4, X3.5
- net VBUS: now also U$23.P, X3.1

Commit message: Block Diagram Update
Parts:
- moved X3 113.3 mm to (8.89, 25.4)
- moved IC1 14.5 mm to (30.5, 26.7)
Changed lines of the file:
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@@
 </autorouter>
 <elements>
-<element name="IC1" library="at90usb" package="TQFP64" value="AT90USB1287-AU" x="39.37" y="38.1"/>
+<element name="IC1" library="at90usb" package="TQFP64" value="AT90USB1287-AU" x="30.48" y="26.67"/>
 <element name="RESET" library="SparkFun-Electromechanical" package="TACTILE_SWITCH_SMD" value="" x="3.81" y="-3.81">
 <attribute name="OC_NEWARK" value="unknown" x="3.81" y="-3.81" size="1.778" layer="27" display="off"/>
@@
 <attribute name="MF" value="" x="2.54" y="-86.36" size="1.778" layer="27" display="off"/>
 </element>
-<element name="X3" library="con-hirose" package="UX60-MB-5S8" value="MINI-USB-UX60-MB-5S8" x="1.27" y="-87.63">
-<attribute name="OC_NEWARK" value="unknown" x="1.27" y="-87.63" size="1.778" layer="27" display="off"/>
-<attribute name="MPN" value="" x="1.27" y="-87.63" size="1.778" layer="27" display="off"/>
-<attribute name="MF" value="" x="1.27" y="-87.63" size="1.778" layer="27" display="off"/>
-<attribute name="OC_FARNELL" value="unknown" x="1.27" y="-87.63" size="1.778" layer="27" display="off"/>
+<element name="X3" library="con-hirose" package="UX60-MB-5S8" value="MINI-USB-UX60-MB-5S8" x="8.89" y="25.4">
+<attribute name="OC_NEWARK" value="unknown" x="8.89" y="25.4" size="1.778" layer="27" display="off"/>
+<attribute name="MPN" value="" x="8.89" y="25.4" size="1.778" layer="27" display="off"/>
+<attribute name="MF" value="" x="8.89" y="25.4" size="1.778" layer="27" display="off"/>
+<attribute name="OC_FARNELL" value="unknown" x="8.89" y="25.4" size="1.778" layer="27" display="off"/>
 </element>
 <element name="R37" library="adafruit" package="R0603" value="22" x="2.54" y="-96.52">
@@
 <contactref element="IC1" pad="6"/>
 <contactref element="C10" pad="2"/>
-<wire x1="9.92" y1="-89.23" x2="3.39" y2="-101.6" width="0" layer="19" extent="1-1"/>
-<wire x1="3.39" y1="-81.28" x2="9.92" y2="-89.23" width="0" layer="19" extent="1-1"/>
+<wire x1="17.54" y1="23.8" x2="3.39" y2="-101.6" width="0" layer="19" extent="1-1"/>
+<wire x1="3.39" y1="-81.28" x2="17.54" y2="23.8" width="0" layer="19" extent="1-1"/>
 <wire x1="6.77" y1="-76.2" x2="3.39" y2="-81.28" width="0" layer="19" extent="1-1"/>
 <wire x1="2.54" y1="-69.85" x2="6.77" y2="-76.2" width="0" layer="19" extent="1-1"/>
@@
 <wire x1="1.27" y1="-5.715" x2="1.27" y2="-18.415" width="0" layer="19" extent="1-1"/>
 <wire x1="6.35" y1="-5.715" x2="1.27" y2="-5.715" width="0" layer="19" extent="1-1"/>
-<wire x1="37.37" y1="30.3" x2="6.35" y2="-5.715" width="0" layer="19" extent="1-1"/>
-<wire x1="31.57" y1="40.1" x2="37.37" y2="30.3" width="0" layer="19" extent="1-1"/>
-<wire x1="34.17" y1="45.9" x2="31.57" y2="40.1" width="0" layer="19" extent="1-1"/>
-<wire x1="42.17" y1="45.9" x2="34.17" y2="45.9" width="0" layer="19" extent="1-1"/>
+<wire x1="28.48" y1="18.87" x2="6.35" y2="-5.715" width="0" layer="19" extent="1-1"/>
+<wire x1="22.68" y1="28.67" x2="28.48" y2="18.87" width="0" layer="19" extent="1-1"/>
+<wire x1="25.28" y1="34.47" x2="22.68" y2="28.67" width="0" layer="19" extent="1-1"/>
+<wire x1="33.28" y1="34.47" x2="25.28" y2="34.47" width="0" layer="19" extent="1-1"/>
 </signal>
 <signal name="VCC">
 <contactref element="IC1" pad="52"/>
 <contactref element="IC1" pad="21"/>
-<wire x1="42.97" y1="45.9" x2="36.57" y2="30.3" width="0" layer="19" extent="1-1"/>
+<wire x1="34.08" y1="34.47" x2="27.68" y2="18.87" width="0" layer="19" extent="1-1"/>
 </signal>
 <signal name="UVCC">
@@
 <contactref element="X3" pad="1"/>
 <contactref element="U$23" pad="P"/>
-<wire x1="9.92" y1="-86.03" x2="13.09" y2="-96.52" width="0" layer="19" extent="1-1"/>
-<wire x1="31.57" y1="38.5" x2="9.92" y2="-86.03" width="0" layer="19" extent="1-1"/>
+<wire x1="17.54" y1="27" x2="13.09" y2="-96.52" width="0" layer="19" extent="1-1"/>
+<wire x1="17.54" y1="27" x2="22.61" y2="27" width="0" layer="19" extent="1-16"/>
+<wire x1="22.61" y1="27" x2="22.68" y2="27.07" width="0.4064" layer="1"/>
 </signal>
 <signal name="3.3V">
@@
 <contactref element="R35" pad="2"/>
 <contactref element="IC1" pad="20"/>
-<wire x1="6.35" y1="-1.905" x2="35.77" y2="30.3" width="0" layer="19" extent="1-1"/>
+<wire x1="6.35" y1="-1.905" x2="26.88" y2="18.87" width="0" layer="19" extent="1-1"/>
 <wire x1="1.27" y1="-1.905" x2="6.35" y2="-1.905" width="0" layer="19" extent="1-1"/>
 <wire x1="3.39" y1="-10.16" x2="1.27" y2="-1.905" width="0" layer="19" extent="1-1"/>
@@
 <contactref element="HWB" pad="1"/>
 <contactref element="IC1" pad="43"/>
-<wire x1="6.35" y1="-14.605" x2="47.17" y2="40.1" width="0" layer="19" extent="1-1"/>
+<wire x1="6.35" y1="-14.605" x2="38.28" y2="28.67" width="0" layer="19" extent="1-1"/>
 <wire x1="1.27" y1="-14.605" x2="6.35" y2="-14.605" width="0" layer="19" extent="1-1"/>
 <wire x1="1.69" y1="-22.86" x2="1.27" y2="-14.605" width="0" layer="19" extent="1-1"/>
@@
 <contactref element="X3" pad="3"/>
 <contactref element="R37" pad="2"/>
-<wire x1="9.92" y1="-87.63" x2="3.39" y2="-96.52" width="0" layer="19" extent="1-1"/>
+<wire x1="17.54" y1="25.4" x2="3.39" y2="-96.52" width="0" layer="19" extent="1-1"/>
 </signal>
 <signal name="N$2">
 <contactref element="X3" pad="2"/>
 <contactref element="R38" pad="2"/>
-<wire x1="9.92" y1="-86.83" x2="8.47" y2="-96.52" width="0" layer="19" extent="1-1"/>
+<wire x1="17.54" y1="26.2" x2="8.47" y2="-96.52" width="0" layer="19" extent="1-1"/>
 </signal>
 <signal name="D-">
@@
 <contactref element="IC1" pad="7"/>
 <contactref element="C10" pad="1"/>
-<wire x1="31.57" y1="39.3" x2="1.69" y2="-101.6" width="0" layer="19" extent="1-1"/>
+<wire x1="22.68" y1="27.87" x2="1.69" y2="-101.6" width="0" layer="19" extent="1-1"/>
 </signal>
 </signals>

Commit message: Update Power Supplies and Library
Parts:
- removed HWB, RESET: (no value), SparkFun-Electromechanical:TACTILE_SWITCH_SMD
- removed X3: MINI-USB-UX60-MB-5S8, con-hirose:UX60-MB-5S8
- added C14: 100nF, SGC:0805
- added C15: 47uF, SGC:1206_190
- added C16, C17: 4.7uF, SGC:C0603
- added C2: 10uF, SparkFun-Capacitors:1210
- added C3, C4: 47uF, SparkFun-Capacitors:EIA3528
- added C5: 10uF, SparkFun-Capacitors:1206
- added C6: 1.0uF, SparkFun-Capacitors:0603-CAP
- added C7: 22uF, SGC:1206_190
- added D1, D2: ZLLS500, SparkFun-DiscreteSemi:SOT23
- added D3: RED, SGC:LED-0603
- added JP2, JP5: M02PTH, SGC:1X02
- added JP3: JUMPER-PTH-2-NC, SparkFun-Passives:PTH-JUMPER-NC_BOTTOM_NO_SILK
- added JP4: R_SEN, SparkFun-Connectors:1X02
- added L1: 68uH, SparkFun-Passives:CR75
- added L2: 1uH, SGC:MLP2520K1R0ST
- added R2: 0.22, SparkFun-Resistors:0805
- added R4, R6: 220k, SparkFun-Resistors:0603-RES
- added R5: 47k, SparkFun-Resistors:0603-RES
- added R7: TRIMPOT, SparkFun-Electromechanical:TRIMPOT-5MM-V2
- added R8: 2.5K, SGC:R0603
- added R9: 330, SGC:R0603
- added U$1: USB_MICRO_B_DX4, SGC:USB_MICRO_B_DX4
- added U$3: TPS63021DSJR, SGC:R-PVSON-N14
- added U1: MCP73831, SGC:SOT23-5
- added U2: LT3652, SparkFun-PowerIC:MSOP-12_GND
- C1: device SparkFun-Capacitors:0603-CAP -> SGC:C0603
- C10, C11, C12, C13, C8, C9: device adafruit:C0603 -> SGC:C0603
- D4, D5: device SparkFun-LED:LED-0603 -> SGC:LED-0603
- IC1: device at90usb:TQFP64 -> SGC:TQFP64
- JP1: device SparkFun-Connectors:1X02 -> SGC:1X02
- R1, R3, R35, R36, R37, R38: device adafruit:R0603 -> SGC:R0603
- R39, R40: device SparkFun-Resistors:0603-RES -> SGC:R0603
- X1: device adafruit:CTS406 -> SGC:CTS406
- moved JP1 82.7 mm to (17.8, 11.4)
Connections:
- removed net ID: X3.4
- new net !CHRG: U2.4
- new net !FAULT: U2.5
- new net BOOST: C6.1, D2.3, U2.11
- new net FB: R4.2, R5.1, R6.2
- new net N$13: D3.A, R9.1
- new net N$14: D3.C, U1.1
- new net N$15: R8.2, U1.5
- new net N$4: R6.1, U2.7
- new net N$5: C3.A, C4.A, C5.1, D2.1, JP3.1, JP4.1, R2.2, R5.2, U2.9
- new net N$6: U$1.ID
- new net N$7: L2.1, U$3.8
- new net N$8: L2.2, U$3.6
- new net N$9: C14.1, U$3.1, U$3.12
- new net NTC: U2.8
- new net SENSE: JP4.2, L1.P$2, R2.1, U2.10
- new net SET: R7.B, U2.2
- new net SOLAR_IN: C2.1, R7.A, U2.1, U2.3
- new net SW: C6.2, D1.3, L1.P$1, U2.12
- new net VBAT: C1.1, C17.1, C7.1, JP1.2, JP3.2, R1.2, U$3.10, U1.3
- net 3.3V: now also C15.1, U$3.3, U$3.4
- net GND: now also C14.2, C15.2, C16.2, C17.2, C2.2, C3.C, C4.C, C5.2, C7.2, D1.1, JP2.2, JP5.2, R4.1, R7.C, R8.1, U$1.GND, U$3.13, U$3.2, U1.2, U2.13, U2.6; no longer HWB.3, HWB.4, RESET.3, RESET.4, X3.5
- net HWB: now also JP5.1; no longer HWB.1, HWB.2
- net N$1: now also U$1.D+; no longer X3.3
- net N$2: now also U$1.D-; no longer X3.2
- net RESET: now also JP2.1; no longer RESET.1, RESET.2
- net VBUS: now also C16.1, R9.2, U$1.VBUS, U1.4; no longer X3.1
- net VIN: no longer C1.1, JP1.2, R1.2

Commit message: Midterm Checkoff
Parts:
- removed C14: 100nF, SGC:0805
- removed C15: 47uF, SGC:1206_190
- removed C7: 22uF, SGC:1206_190
- removed L2: 1uH, SGC:MLP2520K1R0ST
- removed U$23: S1AB-13-F, Helmet:SMB
- added C18, C19, C20, C21: 1.0uF, SGC:C0603
- added J1: POWER_JACKPTH_LOCK, SGC:POWER_JACK_PTH_LOCK
- added JP7: M10LOCK, SGC:1X10_LOCK
- added R10, R11: 4.7K, SGC:R0603
- added U$2, U$4: TPS73633-EP, SGC:SOT23-5
- added U$5, U$8: USB_MICRO_B_DX4, SGC:USB_MICRO_B_DX4
- added U$6: RN4020, SGC:RN4020
- added U$7: SWITCH_SLIDE, SGC:SWITCH_SLIDE
- L1: device SparkFun-Passives:CR75 -> SGC:CR75
- U$3: value TPS63021DSJR -> TPS61030PWPR; device SGC:R-PVSON-N14 -> SGC:TSSOP16
- moved R9 237.1 mm to (8.81, 8.59), flipped to the bottom
- moved D3 231.8 mm to (8.81, 4.04), turned to 270 degrees
- moved U$1 230.1 mm to (-1.27, 20.3), turned to 270 degrees
- moved R8 228.9 mm to (8.81, 4.06), flipped to the bottom
- moved C17 225.4 mm to (11.8, 6.58), flipped to the bottom, turned to 270 degrees
- moved C16 221.2 mm to (8.86, 6.50), flipped to the bottom, turned to 180 degrees
- moved JP2 217.5 mm to (14.9, 25.6)
- moved U1 216.1 mm to (8.61, 6.53), turned to 90 degrees
- moved JP5 208.0 mm to (34.2, 5.08), turned to 270 degrees
- moved U$3 193.7 mm to (78.9, 12.6), turned to 270 degrees
- moved U2 185.3 mm to (70.5, 39.0)
- moved C3 184.7 mm to (66.0, 43.8)
- moved C4 184.7 mm to (74.9, 43.8)
- moved C5 184.7 mm to (76.1, 40.0)
- moved R2 184.7 mm to (81.2, 40.0)
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Connections:
- net N$6 renamed ID
- removed net N$11: C8.1
- removed net N$7: L2.1, U$3.8
- removed net N$8: L2.2, U$3.6
- removed net N$9: C14.1, U$3.1, U$3.12
- removed net VCC: IC1.21, IC1.52
- removed net VIN: U$23.M
- new net BT_CMD: IC1.51, U$6.8
- new net BT_UART_RX: IC1.28, U$6.6
- new net BT_UART_TX: IC1.27, U$6.5
- new net FAN: IC1.50, JP7.3
- new net LBI: U$3.7
- new net MISO: IC1.13, JP7.4
- new net MOSI: IC1.12, JP7.5
- new net N$6: C8.1, IC1.62
- new net SCK: IC1.11, JP7.6
- new net SCL: IC1.25, JP7.9, R11.1
- new net SDA: IC1.26, JP7.8, R10.1
- new net SS: IC1.10, JP7.7
- new net VBAT_IN: C1.1, C17.1, JP1.2, R1.2, U$7.3, U1.3
- new net VBAT_OUT: C20.1, U$4.1, U$4.3, U$7.1
- net 3.3V: now also C19.1, C21.1, IC1.21, IC1.52, JP7.1, R10.2, R11.2, U$2.5, U$4.5, U$6.23; no longer C15.1, U$3.3, U$3.4
- net A6: now also IC1.45
- net A7: now also IC1.44
- net BATTSIG: now also IC1.61
- net D+: now also IC1.5
- net D-: now also IC1.4
- net GND: now also C18.2, C19.2, C20.2, C21.2, J1.GND, J1.GNDBREAK, JP7.2, U$2.2, U$2.4, U$4.2, U$4.4, U$5.GND, U$6.1, U$6.16, U$6.24, U$6.9; no longer C14.2, C15.2, C7.2, U$3.13, U$3.2
- net SOLAR_IN: now also J1.PWR
- net VBAT: now also U$3.6; no longer C1.1, C17.1, C7.1, JP1.2, R1.2, U$3.10, U1.3
- net VBUS: now also C18.1, U$2.1, U$2.3, U$5.VBUS; no longer U$23.P
- net XTAL1: now also IC1.23
- net XTAL2: now also IC1.24
