File: Board Files/SGC.0.sch (EAGLE design)
At the start: 1 part, among them IC1 AT90USB1287-AU

Commit message: Microcontroller block update
Parts:
- added C1: 1.0uF, SparkFun-Capacitors:1.0UF-16V-10%(0603)
- added C10: 1uF, adafruit:C-USC0603
- added C11, C9: 15pF, adafruit:C-USC0603
- added C12, C13, C8: 0.1uF, adafruit:C-USC0603
- added D4, D5: RED, SparkFun-LED:LED-RED0603
- added HWB, RESET: (no value), SparkFun-Electromechanical:TAC_SWITCHSMD
- added JP1: M02PTH, SparkFun-Connectors:M02PTH
- added R1, R3, R35, R36: 47K, adafruit:R-US_R0603
- added R37, R38: 22, adafruit:R-US_R0603
- added R39, R40: 330, SparkFun-Resistors:RESISTOR0603-RES
- added U$23: S1AB-13-F, Helmet:S1AB-13-F
- added X1: (no value), adafruit:CRYSTALCTS406
- added X3: MINI-USB-UX60-MB-5S8, con-hirose:MINI-USB-UX60-MB-5S8
Connections:
- new net 3.3V: C12.1, C13.1, R35.1, R36.2
- new net A6: R39.2
- new net A7: R40.2
- new net BATTSIG: R1.1, R3.2
- new net D+: R37.1
- new net D-: R38.1
- new net GND: C1.2, C10.2, C11.2, C12.2, C13.2, C8.2, C9.2, D4.C, D5.C, HWB.3, HWB.4, IC1.UGND, JP1.1, R3.1, RESET.3, RESET.4, X3.5
- new net HWB: HWB.1, HWB.2, IC1.PE2(ALE/HWB), R36.1
- new net ID: X3.4
- new net N$1: R37.2, X3.3
- new net N$11: C8.1
- new net N$2: R38.2, X3.2
- new net N$29: D4.A, R39.1
- new net N$3: C10.1, IC1.UCAP
- new net N$31: D5.A, R40.1
- new net RESET: IC1.RESET, R35.2, RESET.1, RESET.2
- new net VBUS: U$23.P, X3.1
- new net VIN: C1.1, JP1.2, R1.2, U$23.M
- new net XTAL1: C11.1, X1.1
- new net XTAL2: C9.1, X1.2
Other:
- note added: "8MHZ CRYSTAL"
- note added: "BATTERY INPUT"
- note added: "BOOTLOADER ACTIVATION"
- note added: "MICROCONTROLLER"
- note added: "RESET"

Commit message: Update Power Supplies and Library
Parts:
- removed HWB, RESET: (no value), SparkFun-Electromechanical:TAC_SWITCHSMD
- removed X3: MINI-USB-UX60-MB-5S8, con-hirose:MINI-USB-UX60-MB-5S8
- added C14: 100nF, SGC:08053C104KAT2A
- added C15: 47uF, SGC:GRM31CR60J476ME19L
- added C16, C17: 4.7uF, SGC:C-USC0603
- added C2: 10uF, SparkFun-Capacitors:10UF50V20%(1210)
- added C3, C4: 47uF, SparkFun-Capacitors:47UF-TANT
- added C5: 10uF, SparkFun-Capacitors:10UF-6.3V-20%(1206)
- added C6: 1.0uF, SparkFun-Capacitors:1.0UF-16V-10%(0603)
- added C7: 22uF, SGC:GRM31CR61A226KE19L
- added D1, D2: ZLLS500, SparkFun-DiscreteSemi:ZLLS500ZLLS500
- added D3: RED, SGC:LED0603
- added JP2, JP5: M02PTH, SGC:M02PTH
- added JP3: JUMPER-PTH-2-NC, SparkFun-Passives:JUMPER-PTH-2-NC
- added JP4: R_SEN, SparkFun-Connectors:M02PTH
- added L1: 68uH, SparkFun-Passives:INDUCTOR68UH-1A
- added L2: 1uH, SGC:MLP2520K1R0ST
- added R2: 0.22, SparkFun-Resistors:0.22OHM1/4W1%(0805)
- added R4, R6: 220k, SparkFun-Resistors:220KOHM1/10W1%(0603)
- added R5: 47k, SparkFun-Resistors:47KOHM1/10W1%(0603)
- added R7: TRIMPOT, SparkFun-Electromechanical:TRIMPOT
- added R8: 2.5K, SGC:R-US_R0603
- added R9: 330, SGC:R-US_R0603
- added U$1: USB_MICRO_B_DX4, SGC:USB_MICRO_B_DX4
- added U$3: TPS63021DSJR, SGC:TPS63021DSJR
- added U1: MCP73831, SGC:MCP73831
- added U2: LT3652, SparkFun-PowerIC:LT3652
- C1: device SparkFun-Capacitors:1.0UF-16V-10%(0603) -> SGC:C-USC0603
- C10, C11, C12, C13, C8, C9: device adafruit:C-USC0603 -> SGC:C-USC0603
- D4, D5: device SparkFun-LED:LED-RED0603 -> SGC:LED0603
- IC1: device at90usb:AT90USB1287-AU -> SGC:AT90USB1287-AU
- JP1: device SparkFun-Connectors:M02PTH -> SGC:M02PTH
- R1, R3, R35, R36, R37, R38: device adafruit:R-US_R0603 -> SGC:R-US_R0603
- R39, R40: device SparkFun-Resistors:RESISTOR0603-RES -> SGC:R-US_R0603
- X1: device adafruit:CRYSTALCTS406 -> SGC:CRYSTALCTS406
Connections:
- removed net ID: X3.4
- new net !CHRG: U2.!CHRG
- new net !FAULT: U2.!FAULT
- new net BOOST: C6.1, D2.C, U2.BOOST
- new net FB: R4.2, R5.1, R6.2
- new net N$13: D3.A, R9.1
- new net N$14: D3.C, U1.STAT
- new net N$15: R8.2, U1.PROG
- new net N$4: R6.1, U2.VFB
- new net N$5: C3.+, C4.+, C5.1, D2.A, JP3.1, JP4.1, R2.2, R5.2, U2.BAT
- new net N$6: U$1.P$1
- new net N$7: L2.1, U$3.L1_2
- new net N$8: L2.2, U$3.L2_2
- new net N$9: C14.1, U$3.EN, U$3.VINA
- new net NTC: U2.NTC
- new net SENSE: JP4.2, L1.2, R2.1, U2.SENSE
- new net SET: R7.WIPER, U2.VIN_REG
- new net SOLAR_IN: C2.1, R7.CCW, U2.!SHDN, U2.VIN
- new net SW: C6.2, D1.C, L1.1, U2.SW
- new net VBAT: C1.1, C17.1, C7.1, JP1.2, JP3.2, R1.2, U$3.VIN_2, U1.VBAT
- net 3.3V: now also C15.1, U$3.FB, U$3.VOUT_2
- net GND: now also C14.2, C15.2, C16.2, C17.2, C2.2, C3.-, C4.-, C5.2, C7.2, D1.A, JP2.2, JP5.2, R4.1, R7.CW, R8.1, U$1.4, U$3.GND_2, U$3.PS/SYNC, U1.VSS, U2.GND_PAD, U2.TIMER; no longer HWB.3, HWB.4, RESET.3, RESET.4, X3.5
- net HWB: now also JP5.1; no longer HWB.1, HWB.2
- net N$1: now also U$1.3; no longer X3.3
- net N$2: now also U$1.2; no longer X3.2
- net RESET: now also JP2.1; no longer RESET.1, RESET.2
- net VBUS: now also C16.1, R9.2, U$1.1, U1.VIN; no longer X3.1
- net VIN: no longer C1.1, JP1.2, R1.2
Other:
- note added: "0.22 -> 800mA"
- note added: "0.33 -> 750mA"
- note added: "0.5 -> 650mA"
- note added: "1.0 -> 550mA"
- note added: "3.3V SYSTEM VOLTAGE"
- note added: "Cut the JP3 trace to measure output current. Adjust trim pot until output current reaches its maximum."
- note added: "Ichg = .1/(R1||Rsen)"
- note added: "NOTE: IREG = 1000v / RPROG"
- note added: "NOTE: IREG is set for 400mA charge current"
- note added: "R_SEN is in parallel with R1. Small resistors can be added to increase the charge current from the default ~450mA."
- note added: "SOLAR CHARGER"
- note added: "Typical R_SEN values vs. Ichg"
- note added: "USB BATTERY CHARGER"
- moved on the sheet: C1, R38

Commit message: Midterm Checkoff
Parts:
- removed C14: 100nF, SGC:08053C104KAT2A
- removed C15: 47uF, SGC:GRM31CR60J476ME19L
- removed C7: 22uF, SGC:GRM31CR61A226KE19L
- removed L2: 1uH, SGC:MLP2520K1R0ST
- removed U$23: S1AB-13-F, Helmet:S1AB-13-F
- added C18, C19, C20, C21: 1.0uF, SGC:C-USC0603
- added J1: POWER_JACKPTH_LOCK, SGC:POWER_JACKPTH_LOCK
- added JP7: M10LOCK, SGC:M10LOCK
- added R10, R11: 4.7K, SGC:R-US_R0603
- added U$2, U$4: TPS73633-EP, SGC:TPS73633-EP
- added U$5, U$8: USB_MICRO_B_DX4, SGC:USB_MICRO_B_DX4
- added U$6: RN4020, SGC:RN4020
- added U$7: SWITCH_SLIDE, SGC:SWITCH_SLIDE
- L1: device SparkFun-Passives:INDUCTOR68UH-1A -> SGC:INDUCTOR68UH-1A
- U$3: value TPS63021DSJR -> TPS61030PWPR; device SGC:TPS63021DSJR -> SGC:TPS61030PWPR
Connections:
- net N$6 renamed ID
- removed net N$11: C8.1
- removed net N$7: L2.1, U$3.L1_2
- removed net N$8: L2.2, U$3.L2_2
- removed net N$9: C14.1, U$3.EN, U$3.VINA
- removed net VIN: U$23.M
- new net BT_CMD: IC1.PA0(AD0), U$6.CMD/MLDP
- new net BT_UART_RX: IC1.PD3(TXD1/INT3), U$6.UART_RX
- new net BT_UART_TX: IC1.PD2(RXD1/INT2), U$6.UART_TX
- new net FAN: IC1.PA1(AD1), JP7.3
- new net MISO: IC1.PB3(PDO/PCINT3/MISO), JP7.4
- new net MOSI: IC1.PB2(PDI/PCINT2/MOSI), JP7.5
- new net N$6: C8.1, IC1.AREF
- new net SCK: IC1.PB1(PCINT1/SCK), JP7.6
- new net SCL: IC1.PD0(OC.0B/SCL/INT0), JP7.9, R11.1
- new net SDA: IC1.PD1(OC.2B/SDA/INT1), JP7.8, R10.1
- new net SS: IC1.PB0(SS/PCINT0), JP7.7
- new net VBAT_IN: C1.1, C17.1, JP1.2, R1.2, U$7.@3, U1.VBAT
- new net VBAT_OUT: C20.1, U$4.@VIN, U$7.@1
- net 3.3V: now also C19.1, C21.1, IC1.VCC@1, IC1.VCC@2, JP7.1, R10.2, R11.2, U$2.@VOUT, U$4.@VOUT, U$6.VDD; no longer C15.1, U$3.FB, U$3.VOUT_2
- net A6: now also IC1.PA6(AD6)
- net A7: now also IC1.PA7(AD7)
- net BATTSIG: now also IC1.PF0(ADC0)
- net D+: now also IC1.D+
- net D-: now also IC1.D-
- net GND: now also C18.2, C19.2, C20.2, C21.2, J1.GND, J1.GNDBREAK, JP7.2, U$2.@GND, U$4.@GND, U$5.4, U$6.GND0, U$6.GND1, U$6.GND2, U$6.GND3; no longer C14.2, C15.2, C7.2, U$3.GND_2, U$3.PS/SYNC
- net SOLAR_IN: now also J1.PWR
- net VBAT: no longer C1.1, C17.1, C7.1, JP1.2, R1.2, U$3.VIN_2, U1.VBAT
- net VBUS: now also C18.1, U$2.@VIN, U$5.1; no longer U$23.P
- net XTAL1: now also IC1.XTAL2
- net XTAL2: now also IC1.XTAL1
Other:
- note added: "BLUETOOTH"
- note added: "FLASH UTILITY"
- moved on the sheet: C16, C17, D3, R37, R38, R8, R9, U1
